File: hardware/hyperion.kicad_pcb (KiCad board)
At the start: 2 copper layers, 34 x 28 mm, 90 parts, among them Q1 AON7403, U1 RP2354A, U2 DRV8231ADSGR, U3 DRV8231ADSGR, U4 LMR51610YDBVR, U5 ME6211C33M5G, U6 LSM6DSV32XTR, Y1 12MHz ABM8-272-T3

Commit message: WIP snapshot from zlaticko 2026-11-01
Co-Authored-By: Claude Opus 5.5 <noreply@anthropic.com>
Parts:
- R13, R14: value 1.1k 1% -> 1.5k 1%
Changed lines of the file:
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@@
 			)
 		)
-		(property "Value" "1.1k 1%"
+		(property "Value" "1.5k 1%"
 			(at 0 1.43 90)
 			(layer "F.Fab")
@@
 			)
 		)
-		(property "LCSC" "C22764"
+		(property "LCSC" "C22843"
 			(at 0 0 90)
 			(unlocked yes)
@@
 			)
 		)
-		(property "MPN" "0603WAF1101T5E"
+		(property "MPN" "0603WAF1501T5E"
 			(at 0 0 90)
 			(unlocked yes)
@@
 			)
 		)
-		(property "Value" "1.1k 1%"
+		(property "Value" "1.5k 1%"
 			(at 0 1.43 0)
 			(layer "F.Fab")
@@
 			)
 		)
-		(property "LCSC" "C22764"
+		(property "LCSC" "C22843"
 			(at 0 0 0)
 			(unlocked yes)
@@
 			)
 		)
-		(property "MPN" "0603WAF1101T5E"
+		(property "MPN" "0603WAF1501T5E"
 			(at 0 0 0)
 			(unlocked yes)
@@
 	)
 	(gr_poly
+		(pts
+			(xy 127.475 104.899999) (xy 127.473838 104.923004) (xy 127.470428 104.945345) (xy 127.464884 104.966908)
+			(xy 127.457318 104.98758) (xy 127.447843 105.007248) (xy 127.436573 105.025799) (xy 127.42362 105.04312)
+			(xy 127.409099 105.059099) (xy 127.39312 105.07362) (xy 127.375799 105.086573) (xy 127.357248 105.097843)
+			(xy 127.33758 105.107318) (xy 127.316908 105.114884) (xy 127.295345 105.120428) (xy 127.273004 105.123838)
+			(xy 127.25 105.125) (xy 127.226995 105.123838) (xy 127.204654 105.120428) (xy 127.183091 105.114884)
+			(xy 127.162419 105.107318) (xy 127.142751 105.097843) (xy 127.1242 105.086573) (xy 127.106879 105.07362)
+			(xy 127.0909 105.059099) (xy 127.076379 105.04312) (xy 127.063426 105.025799) (xy 127.052156 105.007248)
+			(xy 127.042681 104.98758) (xy 127.035115 104.966908) (xy 127.029571 104.945345) (xy 127.026161 104.923004)
+			(xy 127.025 104.899999) (xy 127.026161 104.876995) (xy 127.029571 104.854654) (xy 127.035115 104.833091)
+			(xy 127.042681 104.812419) (xy 127.052156 104.792751) (xy 127.063426 104.7742) (xy 127.076379 104.756879)
+			(xy 127.0909 104.7409) (xy 127.106879 104.726379) (xy 127.1242 104.713426) (xy 127.142751 104.702156)
+			(xy 127.162419 104.692681) (xy 127.183091 104.685115) (xy 127.204654 104.679571) (xy 127.226995 104.676161)
+			(xy 127.25 104.675) (xy 127.273004 104.676161) (xy 127.295345 104.679571) (xy 127.316908 104.685115)
+			(xy 127.33758 104.692681) (xy 127.357248 104.702156) (xy 127.375799 104.713426) (xy 127.39312 104.726379)
+			(xy 127.409099 104.7409) (xy 127.42362 104.756879) (xy 127.436573 104.7742) (xy 127.447843 104.792751)
+			(xy 127.457318 104.812419) (xy 127.464884 104.833091) (xy 127.470428 104.854654) (xy 127.473838 104.876995)
+		)
+		(stroke
+			(width 0)
+			(type default)
+		)
+		(fill yes)
+		(layer "F.SilkS")
+	)
+	(gr_poly
