File: hardware/motors.kicad_sch (KiCad schematic)
At the start: 12 parts, among them U2 DRV8231ADSGR, U3 DRV8231ADSGR

Commit message: WIP snapshot from zlaticko 2026-11-01
Co-Authored-By: Claude Opus 5.5 <noreply@anthropic.com>
Parts:
- R13, R14: value 1.1k 1% -> 1.5k 1%; LCSC C22764 -> C22843; MPN 0603WAF1101T5E -> 0603WAF1501T5E
Changed lines of the file:
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@@
 			)
 		)
-		(property "Value" "1.1k 1%"
+		(property "Value" "1.5k 1%"
 			(at 132.08 81.28 90)
 			(effects
@@
 			)
 		)
-		(property "LCSC" "C22764"
+		(property "LCSC" "C22843"
 			(at 132.08 81.28 0)
 			(hide yes)
@@
 			)
 		)
-		(property "MPN" "0603WAF1101T5E"
+		(property "MPN" "0603WAF1501T5E"
 			(at 132.08 81.28 0)
 			(hide yes)
@@
 			)
 		)
-		(property "Value" "1.1k 1%"
+		(property "Value" "1.5k 1%"
 			(at 132.08 154.94 90)
 			(effects
@@
 			)
 		)
-		(property "LCSC" "C22764"
+		(property "LCSC" "C22843"
 			(at 132.08 154.94 0)
 			(hide yes)
@@
 			)
 		)
-		(property "MPN" "0603WAF1101T5E"
+		(property "MPN" "0603WAF1501T5E"
 			(at 132.08 154.94 0)
 			(hide yes)
